Commit message: Add socket timeout to ros2 control macro

File: kuka_kr16_support/robots/kr16_2.urdf.xacro (robot description, xacro)
@@ -4,4 +4,5 @@
   <xacro:arg name="rsi_ip" default="127.0.0.1"/>
   <xacro:arg name="rsi_port" default="49152"/>
+  <xacro:arg name="socket_timeout" default="30.0"/>
   <xacro:arg name="load_ros2_control" default="false"/>
   <xacro:arg name="connected_to" default=""/>
@@ -17,4 +18,5 @@
             rsi_ip="$(arg rsi_ip)"
             rsi_port="$(arg rsi_port)"
+            rsi_timeout="$(arg socket_timeout)"
     />
   </xacro:if>

File: kuka_kr16_support/ros2_control/kr16_2.ros2_control.xacro (robot description, xacro)
@@ -1,5 +1,5 @@
 <?xml version="1.0"?>
 <robot xmlns:xacro="http://www.ros.org/wiki/xacro" name="kr16_2_ros2_control">
-  <xacro:macro name="kr16_2_interface" params="name prefix rsi_ip rsi_port">
+  <xacro:macro name="kr16_2_interface" params="name prefix rsi_ip rsi_port socket_timeout">
     <ros2_control name="${name}" type="system">
       <hardware>
@@ -7,4 +7,5 @@
         <param name="rsi_ip">${rsi_ip}</param>
         <param name="rsi_port">${rsi_port}</param>
+        <param name="socket_timeout">${socket_timeout}</param>
       </hardware>
       <joint name="${prefix}joint_a1">

Commit message: Add KR16 description (#3)
* Add kr16 meshes

* Add kr16 xacro macros

* Small fixes in kr16_2 macros

* KR16 as default

File: kuka_kr16_support/robots/kr16_2.urdf.xacro (robot description, xacro)
@@ -18,5 +18,5 @@
             rsi_ip="$(arg rsi_ip)"
             rsi_port="$(arg rsi_port)"
-            rsi_timeout="$(arg socket_timeout)"
+            socket_timeout="$(arg socket_timeout)"
     />
   </xacro:if>

File: kuka_kr16_support/robots/kr16_2.xacro (robot description, xacro)
@@ -204,5 +204,4 @@
     <!-- END JOINTS -->
     <xacro:if value="${connected_to == ''}">
-      <link name="world"/>
       <xacro:property name="base_frame_name" value="world"/>
     </xacro:if>
@@ -210,4 +209,5 @@
       <xacro:property name="base_frame_name" value="${connected_to}"/>
     </xacro:unless>
+    <link name="${base_frame_name}"/>
     <joint name="${base_frame_name}-${prefix}base_link" type="fixed">
       <origin xyz="${xyz}" rpy="${rpy}"/>
