Commit message: Add KR16 sensor state interfaces to ros2 control macro (#5)
* Add sensor state interfaces to ros2 control macro

* Mock FT sensor data in simulator

* 1D numpy array

File: kuka_kr16_support/robots/kr16.urdf.xacro (robot description, xacro)
@@ -5,4 +5,5 @@
   <xacro:arg name="rsi_port" default="49152"/>
   <xacro:arg name="socket_timeout" default="30"/>
+  <xacro:arg name="has_ft_sensor" default="false"/>
   <xacro:arg name="load_ros2_control" default="false"/>
   <xacro:arg name="connected_to" default=""/>
@@ -10,7 +11,7 @@
   <xacro:arg name="rpy" default="0 0 0"/>
   <xacro:include filename="$(find kuka_kr16_support)/robots/kr16.xacro"/>
-  <xacro:include filename="$(find kuka_kr16_support)/ros2_control/kr16.ros2_control.xacro"/>
   <xacro:kr16 prefix="$(arg prefix)" connected_to="$(arg connected_to)" xyz="$(arg xyz)" rpy="$(arg rpy)"/>
   <xacro:if value="$(arg load_ros2_control)">
+    <xacro:include filename="$(find kuka_kr16_support)/ros2_control/kr16.ros2_control.xacro"/>
     <xacro:kr16_interface
             name="RsiInterface"
@@ -19,4 +20,5 @@
             rsi_port="$(arg rsi_port)"
             socket_timeout="$(arg socket_timeout)"
+            has_ft_sensor="$(arg has_ft_sensor)"
     />
   </xacro:if>

File: kuka_kr16_support/ros2_control/kr16.ros2_control.xacro (robot description, xacro)
@@ -1,5 +1,5 @@
 <?xml version="1.0"?>
 <robot xmlns:xacro="http://www.ros.org/wiki/xacro" name="kr16_ros2_control">
-  <xacro:macro name="kr16_interface" params="name prefix rsi_ip rsi_port socket_timeout">
+  <xacro:macro name="kr16_interface" params="name prefix rsi_ip rsi_port socket_timeout has_ft_sensor">
     <ros2_control name="${name}" type="system">
       <hardware>
@@ -75,4 +75,14 @@
         <state_interface name="position"/>
       </joint>
+      <xacro:if value="${has_ft_sensor}">
+        <sensor name="${prefix}ft_sensor">
+          <state_interface name="force.x"/>
+          <state_interface name="force.y"/>
+          <state_interface name="force.z"/>
+          <state_interface name="torque.x"/>
+          <state_interface name="torque.y"/>
+          <state_interface name="torque.z"/>
+        </sensor>
+      </xacro:if>
     </ros2_control>
   </xacro:macro>
