Commit message: Migrate kuka_kr16_support package to ros2 (#2)
* Update CMakeLists and package.xml to ros2

* Delete ros files

* Update xacro macros to match AICA style

* Add ros2 control macro

* Add launch file and rviz config for visualization

* Add velocity command interface

* Add socket timeout to ros2 control macro

* Socket timeout should be int

File: kuka_kr16_support/urdf/kr16_2.urdf (robot description, URDF)
Before this commit: robot kuka_kr16_2, 9 links, 8 joints
Links:
- removed link base
- removed link base_link
- removed link link_1
- removed link link_2
- removed link link_3
- removed link link_4
- removed link link_5
- removed link link_6
- removed link tool0
- added link kr16_2_base
- added link kr16_2_base_link, mass 2; collision mesh filename=package://kuka_kr16_support/meshes/kr16_2/collision/base_li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; visual mesh filename=package://kuka_kr16_support/meshes/kr16_2/visual/base_link.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
- added link kr16_2_flange
- added link kr16_2_link_1, mass 2; collision mesh filename=package://kuka_kr16_support/meshes/kr16_2/collision/link_1.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; visual mesh filename=package://kuka_kr16_support/meshes/kr16_2/visual/link_1.dae
- added link kr16_2_link_2, mass 2; collision mesh filename=package://kuka_kr16_support/meshes/kr16_2/collision/link_2.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; visual mesh filename=package://kuka_kr16_support/meshes/kr16_2/visual/link_2.dae
- added link kr16_2_link_3, mass 2; collision mesh filename=package://kuka_kr16_support/meshes/kr16_2/collision/link_3.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; visual mesh filename=package://kuka_kr16_support/meshes/kr16_2/visual/link_3.dae
- added link kr16_2_link_4, mass 2; collision mesh filename=package://kuka_kr16_support/meshes/kr16_2/collision/link_4.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; visual mesh filename=package://kuka_kr16_support/meshes/kr16_2/visual/link_4.dae
- added link kr16_2_link_5, mass 2; collision mesh filename=package://kuka_kr16_support/meshes/kr16_2/collision/link_5.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; visual mesh filename=package://kuka_kr16_support/meshes/kr16_2/visual/link_5.dae
- added link kr16_2_link_6, mass 2; collision mesh filename=package://kuka_kr16_support/meshes/kr16_2/collision/link_6.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; visual mesh filename=package://kuka_kr16_support/meshes/kr16_2/visual/link_6.dae
- added link kr16_2_tool0
- added link world
Joints:
- removed joint base_link-base
- removed joint joint_a1
- removed joint joint_a2
- removed joint joint_a3
- removed joint joint_a4
- removed joint joint_a5
- removed joint joint_a6
- removed joint joint_a6-tool0
- added joint kr16_2_base_link-base: type fixed, parent kr16_2_base_link, child kr16_2_base, origin xyz=0 0 0 rpy=0 0 0
- added joint kr16_2_flange-tool0: type fixed, parent kr16_2_flange, child kr16_2_tool0, origin xyz=0 0 0 rpy=0 1.5707963267948966 0
- added joint kr16_2_joint_a1: type revolute, parent kr16_2_base_link, child kr16_2_link_1, origin xyz=0 0 0.675 rpy=0 0 0, axis 0 0 -1, limit lower=-3.2288591161895095 upper=3.2288591161895095 effort=0 velocity=2.722713633111154
- added joint kr16_2_joint_a2: type revolute, parent kr16_2_link_1, child kr16_2_link_2, origin xyz=0.26 0 0 rpy=0 0 0, axis 0 1 0, limit lower=-2.705260340591211 upper=0.6108652381980153 effort=0 velocity=2.722713633111154
- added joint kr16_2_joint_a3: type revolute, parent kr16_2_link_2, child kr16_2_link_3, origin xyz=0.68 0 0 rpy=0 0 0, axis 0 1 0, limit lower=-2.2689280275926285 upper=2.6878070480712677 effort=0 velocity=2.722713633111154
- added joint kr16_2_joint_a4: type revolute, parent kr16_2_link_3, child kr16_2_link_4, origin xyz=0.67 0 -0.035 rpy=0 0 0, axis -1 0 0, limit lower=-6.1086523819801535 upper=6.1086523819801535 effort=0 velocity=5.759586531581287
- added joint kr16_2_joint_a5: type revolute, parent kr16_2_link_4, child kr16_2_link_5, origin xyz=0 0 0 rpy=0 0 0, axis 0 1 0, limit lower=-2.2689280275926285 upper=2.2689280275926285 effort=0 velocity=5.759586531581287
- added joint kr16_2_joint_a6: type revolute, parent kr16_2_link_5, child kr16_2_link_6, origin xyz=0 0 0 rpy=0 0 0, axis -1 0 0, limit lower=-6.1086523819801535 upper=6.1086523819801535 effort=0 velocity=10.733774899765127
- added joint kr16_2_joint_a6-flange: type fixed, parent kr16_2_link_6, child kr16_2_flange, origin xyz=0.158 0 0 rpy=0 0 0
- added joint world-kr16_2_base_link: type fixed, parent world, child kr16_2_base_link, origin xyz=0 0 0 rpy=0 0 0
