Commit message: refactor: rename package to kuka_kr_description

File: kuka_kr_description/robots/kr16.urdf.xacro (robot description, xacro)
@@ -10,8 +10,8 @@
   <xacro:arg name="xyz" default="0 0 0"/>
   <xacro:arg name="rpy" default="0 0 0"/>
-  <xacro:include filename="$(find kuka_kr16_support)/robots/kr16.xacro"/>
+  <xacro:include filename="$(find kuka_kr_description)/robots/kr16.xacro"/>
   <xacro:kr16 prefix="$(arg prefix)" connected_to="$(arg connected_to)" xyz="$(arg xyz)" rpy="$(arg rpy)"/>
   <xacro:if value="$(arg load_ros2_control)">
-    <xacro:include filename="$(find kuka_kr16_support)/ros2_control/kr16.ros2_control.xacro"/>
+    <xacro:include filename="$(find kuka_kr_description)/ros2_control/kr16.ros2_control.xacro"/>
     <xacro:kr16_interface
             name="RsiInterface"

File: kuka_kr_description/robots/kr16.xacro (robot description, xacro)
@@ -8,5 +8,5 @@
         <origin xyz="0 0 0" rpy="0 0 0"/>
         <geometry>
-          <mesh filename="package://kuka_kr16_support/meshes/kr16/visual/base_link.dae" />
+          <mesh filename="package://kuka_kr_description/meshes/kr16/visual/base_link.dae" />
         </geometry>
       </visual>
@@ -17,5 +17,5 @@
         <origin xyz="0 0 0" rpy="0 0 0"/>
         <geometry>
-          <mesh filename="package://kuka_kr16_support/meshes/kr16/visual/link_1.dae" />
+          <mesh filename="package://kuka_kr_description/meshes/kr16/visual/link_1.dae" />
         </geometry>
       </visual>
@@ -26,5 +26,5 @@
         <origin xyz="0 0 0" rpy="0 0 0"/>
         <geometry>
-          <mesh filename="package://kuka_kr16_support/meshes/kr16/visual/link_2.dae"/>
+          <mesh filename="package://kuka_kr_description/meshes/kr16/visual/link_2.dae"/>
         </geometry>
       </visual>
@@ -35,5 +35,5 @@
         <origin xyz="0 0 0" rpy="0 0 0"/>
         <geometry>
-          <mesh filename="package://kuka_kr16_support/meshes/kr16/visual/link_3.dae" />
+          <mesh filename="package://kuka_kr_description/meshes/kr16/visual/link_3.dae" />
         </geometry>
       </visual>
@@ -44,5 +44,5 @@
         <origin xyz="0 0 0" rpy="0 0 0"/>
         <geometry>
-          <mesh filename="package://kuka_kr16_support/meshes/kr16/visual/link_4.dae" />
+          <mesh filename="package://kuka_kr_description/meshes/kr16/visual/link_4.dae" />
         </geometry>
       </visual>
@@ -53,5 +53,5 @@
         <origin xyz="0 0 0" rpy="0 0 0"/>
         <geometry>
-          <mesh filename="package://kuka_kr16_support/meshes/kr16/visual/link_5.dae" />
+          <mesh filename="package://kuka_kr_description/meshes/kr16/visual/link_5.dae" />
         </geometry>
       </visual>
@@ -62,5 +62,5 @@
         <origin xyz="0 0 0" rpy="0 0 0"/>
         <geometry>
-          <mesh filename="package://kuka_kr16_support/meshes/kr16/visual/link_6.dae" />
+          <mesh filename="package://kuka_kr_description/meshes/kr16/visual/link_6.dae" />
         </geometry>
       </visual>

File: kuka_kr_description/robots/kr16_2.urdf.xacro (robot description, xacro)
@@ -9,6 +9,6 @@
   <xacro:arg name="xyz" default="0 0 0"/>
   <xacro:arg name="rpy" default="0 0 0"/>
-  <xacro:include filename="$(find kuka_kr16_support)/robots/kr16_2.xacro"/>
-  <xacro:include filename="$(find kuka_kr16_support)/ros2_control/kr16_2.ros2_control.xacro"/>
+  <xacro:include filename="$(find kuka_kr_description)/robots/kr16_2.xacro"/>
+  <xacro:include filename="$(find kuka_kr_description)/ros2_control/kr16_2.ros2_control.xacro"/>
   <xacro:kr16_2 prefix="$(arg prefix)" connected_to="$(arg connected_to)" xyz="$(arg xyz)" rpy="$(arg rpy)"/>
   <xacro:if value="$(arg load_ros2_control)">

File: kuka_kr_description/robots/kr16_2.xacro (robot description, xacro)
@@ -13,11 +13,11 @@
         <origin xyz="0 0 0" rpy="0 0 0"/>
         <geometry>
-          <mesh filename="package://kuka_kr16_support/meshes/kr16_2/visual/base_link.dae" />
-        </geometry>
-      </visual>
-      <collision>
-        <origin xyz="0 0 0" rpy="0 0 0"/>
-        <geometry>
-          <mesh filename="package://kuka_kr16_support/meshes/kr16_2/collision/base_link.stl" />
+          <mesh filename="package://kuka_kr_description/meshes/kr16_2/visual/base_link.dae" />
+        </geometry>
+      </visual>
+      <collision>
+        <origin xyz="0 0 0" rpy="0 0 0"/>
+        <geometry>
+          <mesh filename="package://kuka_kr_description/meshes/kr16_2/collision/base_link.stl" />
         </geometry>
       </collision>
@@ -33,11 +33,11 @@
         <origin xyz="0 0 0" rpy="0 0 0"/>
         <geometry>
-          <mesh filename="package://kuka_kr16_support/meshes/kr16_2/visual/link_1.dae" />
-        </geometry>
-      </visual>
-      <collision>
-        <origin xyz="0 0 0" rpy="0 0 0"/>
-        <geometry>
-          <mesh filename="package://kuka_kr16_support/meshes/kr16_2/collision/link_1.stl" />
+          <mesh filename="package://kuka_kr_description/meshes/kr16_2/visual/link_1.dae" />
+        </geometry>
+      </visual>
+      <collision>
+        <origin xyz="0 0 0" rpy="0 0 0"/>
+        <geometry>
+          <mesh filename="package://kuka_kr_description/meshes/kr16_2/collision/link_1.stl" />
         </geometry>
       </collision>
@@ -53,11 +53,11 @@
         <origin xyz="0 0 0" rpy="0 0 0"/>
         <geometry>
-          <mesh filename="package://kuka_kr16_support/meshes/kr16_2/visual/link_2.dae"/>
-        </geometry>
-      </visual>
-      <collision>
-        <origin xyz="0 0 0" rpy="0 0 0"/>
-        <geometry>
-          <mesh filename="package://kuka_kr16_support/meshes/kr16_2/collision/link_2.stl" />
+          <mesh filename="package://kuka_kr_description/meshes/kr16_2/visual/link_2.dae"/>
+        </geometry>
+      </visual>
+      <collision>
+        <origin xyz="0 0 0" rpy="0 0 0"/>
+        <geometry>
+          <mesh filename="package://kuka_kr_description/meshes/kr16_2/collision/link_2.stl" />
         </geometry>
       </collision>
@@ -73,11 +73,11 @@
         <origin xyz="0 0 0" rpy="0 0 0"/>
         <geometry>
-          <mesh filename="package://kuka_kr16_support/meshes/kr16_2/visual/link_3.dae" />
-        </geometry>
-      </visual>
-      <collision>
-        <origin xyz="0 0 0" rpy="0 0 0"/>
-        <geometry>
-          <mesh filename="package://kuka_kr16_support/meshes/kr16_2/collision/link_3.stl" />
+          <mesh filename="package://kuka_kr_description/meshes/kr16_2/visual/link_3.dae" />
+        </geometry>
+      </visual>
+      <collision>
+        <origin xyz="0 0 0" rpy="0 0 0"/>
+        <geometry>
+          <mesh filename="package://kuka_kr_description/meshes/kr16_2/collision/link_3.stl" />
         </geometry>
       </collision>
@@ -93,11 +93,11 @@
         <origin xyz="0 0 0" rpy="0 0 0"/>
         <geometry>
-          <mesh filename="package://kuka_kr16_support/meshes/kr16_2/visual/link_4.dae" />
-        </geometry>
-      </visual>
-      <collision>
-        <origin xyz="0 0 0" rpy="0 0 0"/>
-        <geometry>
-          <mesh filename="package://kuka_kr16_support/meshes/kr16_2/collision/link_4.stl" />
+          <mesh filename="package://kuka_kr_description/meshes/kr16_2/visual/link_4.dae" />
+        </geometry>
+      </visual>
+      <collision>
+        <origin xyz="0 0 0" rpy="0 0 0"/>
+        <geometry>
+          <mesh filename="package://kuka_kr_description/meshes/kr16_2/collision/link_4.stl" />
         </geometry>
       </collision>
@@ -113,11 +113,11 @@
         <origin xyz="0 0 0" rpy="0 0 0"/>
         <geometry>
-          <mesh filename="package://kuka_kr16_support/meshes/kr16_2/visual/link_5.dae" />
-        </geometry>
-      </visual>
-      <collision>
-        <origin xyz="0 0 0" rpy="0 0 0"/>
-        <geometry>
-          <mesh filename="package://kuka_kr16_support/meshes/kr16_2/collision/link_5.stl" />
+          <mesh filename="package://kuka_kr_description/meshes/kr16_2/visual/link_5.dae" />
+        </geometry>
+      </visual>
+      <collision>
+        <origin xyz="0 0 0" rpy="0 0 0"/>
+        <geometry>
+          <mesh filename="package://kuka_kr_description/meshes/kr16_2/collision/link_5.stl" />
         </geometry>
       </collision>
@@ -133,11 +133,11 @@
         <origin xyz="0 0 0" rpy="0 0 0"/>
         <geometry>
-          <mesh filename="package://kuka_kr16_support/meshes/kr16_2/visual/link_6.dae" />
-        </geometry>
-      </visual>
-      <collision>
-        <origin xyz="0 0 0" rpy="0 0 0"/>
-        <geometry>
-          <mesh filename="package://kuka_kr16_support/meshes/kr16_2/collision/link_6.stl" />
+          <mesh filename="package://kuka_kr_description/meshes/kr16_2/visual/link_6.dae" />
+        </geometry>
+      </visual>
+      <collision>
+        <origin xyz="0 0 0" rpy="0 0 0"/>
+        <geometry>
+          <mesh filename="package://kuka_kr_description/meshes/kr16_2/collision/link_6.stl" />
         </geometry>
       </collision>
