Commit message: fix: package paths

File: kuka_kr_description/robots/kr70.urdf.xacro (robot description, xacro)
@@ -10,8 +10,8 @@
   <xacro:arg name="xyz" default="0 0 0"/>
   <xacro:arg name="rpy" default="0 0 0"/>
-  <xacro:include filename="$(find kuka_kr70_support)/robots/kr70.xacro"/>
+  <xacro:include filename="$(find kuka_kr_description)/robots/kr70.xacro"/>
   <xacro:kr16 prefix="$(arg prefix)" connected_to="$(arg connected_to)" xyz="$(arg xyz)" rpy="$(arg rpy)"/>
   <xacro:if value="$(arg load_ros2_control)">
-    <xacro:include filename="$(find kuka_kr70_support)/ros2_control/kr70.ros2_control.xacro"/>
+    <xacro:include filename="$(find kuka_kr_description)/ros2_control/kr70.ros2_control.xacro"/>
     <xacro:kr16_interface
             name="RsiInterface"

File: kuka_kr_description/robots/kr70.xacro (robot description, xacro)
@@ -8,5 +8,5 @@
         <origin xyz="0 0 0" rpy="0 0 0"/>
         <geometry>
-          <mesh filename="package://kuka_kr70_support/meshes/kr70/visual/base_link.dae" />
+          <mesh filename="package://kuka_kr_description/meshes/kr70/visual/base_link.dae" />
         </geometry>
       </visual>
@@ -17,5 +17,5 @@
         <origin xyz="0 0 0" rpy="0 0 0"/>
         <geometry>
-          <mesh filename="package://kuka_kr70_support/meshes/kr70/visual/link_1.dae" />
+          <mesh filename="package://kuka_kr_description/meshes/kr70/visual/link_1.dae" />
         </geometry>
       </visual>
@@ -26,5 +26,5 @@
         <origin xyz="0 0 0" rpy="0 0 0"/>
         <geometry>
-          <mesh filename="package://kuka_kr70_support/meshes/kr70/visual/link_2.dae"/>
+          <mesh filename="package://kuka_kr_description/meshes/kr70/visual/link_2.dae"/>
         </geometry>
       </visual>
@@ -35,5 +35,5 @@
         <origin xyz="0 0 0" rpy="0 0 0"/>
         <geometry>
-          <mesh filename="package://kuka_kr70_support/meshes/kr70/visual/link_3.dae" />
+          <mesh filename="package://kuka_kr_description/meshes/kr70/visual/link_3.dae" />
         </geometry>
       </visual>
@@ -44,5 +44,5 @@
         <origin xyz="0 0 0" rpy="0 0 0"/>
         <geometry>
-          <mesh filename="package://kuka_kr70_support/meshes/kr70/visual/link_4.dae" />
+          <mesh filename="package://kuka_kr_description/meshes/kr70/visual/link_4.dae" />
         </geometry>
       </visual>
@@ -53,5 +53,5 @@
         <origin xyz="0 0 0" rpy="0 0 0"/>
         <geometry>
-          <mesh filename="package://kuka_kr70_support/meshes/kr70/visual/link_5.dae" />
+          <mesh filename="package://kuka_kr_description/meshes/kr70/visual/link_5.dae" />
         </geometry>
       </visual>
@@ -62,5 +62,5 @@
         <origin xyz="0 0 0" rpy="0 0 0"/>
         <geometry>
-          <mesh filename="package://kuka_kr70_support/meshes/kr70/visual/link_6.dae" />
+          <mesh filename="package://kuka_kr_description/meshes/kr70/visual/link_6.dae" />
         </geometry>
       </visual>
