Commit message: feat!: update ros2 control macro

File: kuka_kr_description/robots/kr10_r1100_2.urdf.xacro (robot description, xacro)
@@ -4,5 +4,6 @@
   <xacro:arg name="rsi_ip" default="127.0.0.1"/>
   <xacro:arg name="rsi_port" default="49152"/>
-  <xacro:arg name="socket_timeout" default="30"/>
+  <xacro:arg name="connection_timeout" default="30"/>
+  <xacro:arg name="communication_timeout" default="1"/>
   <xacro:arg name="has_ft_sensor" default="false"/>
   <xacro:arg name="load_ros2_control" default="false"/>
@@ -19,5 +20,6 @@
             rsi_ip="$(arg rsi_ip)"
             rsi_port="$(arg rsi_port)"
-            socket_timeout="$(arg socket_timeout)"
+            connection_timeout="$(arg connection_timeout)"
+            communication_timeout="$(arg communication_timeout)"
             has_ft_sensor="$(arg has_ft_sensor)"
     />

File: kuka_kr_description/robots/kr16.urdf.xacro (robot description, xacro)
@@ -4,5 +4,6 @@
   <xacro:arg name="rsi_ip" default="127.0.0.1"/>
   <xacro:arg name="rsi_port" default="49152"/>
-  <xacro:arg name="socket_timeout" default="30"/>
+  <xacro:arg name="connection_timeout" default="30"/>
+  <xacro:arg name="communication_timeout" default="1"/>
   <xacro:arg name="has_ft_sensor" default="false"/>
   <xacro:arg name="load_ros2_control" default="false"/>
@@ -19,5 +20,6 @@
             rsi_ip="$(arg rsi_ip)"
             rsi_port="$(arg rsi_port)"
-            socket_timeout="$(arg socket_timeout)"
+            connection_timeout="$(arg connection_timeout)"
+            communication_timeout="$(arg communication_timeout)"
             has_ft_sensor="$(arg has_ft_sensor)"
     />

File: kuka_kr_description/robots/kr16_2.urdf.xacro (robot description, xacro)
@@ -4,5 +4,6 @@
   <xacro:arg name="rsi_ip" default="127.0.0.1"/>
   <xacro:arg name="rsi_port" default="49152"/>
-  <xacro:arg name="socket_timeout" default="30"/>
+  <xacro:arg name="connection_timeout" default="30"/>
+  <xacro:arg name="communication_timeout" default="1"/>
   <xacro:arg name="load_ros2_control" default="false"/>
   <xacro:arg name="connected_to" default=""/>
@@ -18,5 +19,6 @@
             rsi_ip="$(arg rsi_ip)"
             rsi_port="$(arg rsi_port)"
-            socket_timeout="$(arg socket_timeout)"
+            connection_timeout="$(arg connection_timeout)"
+            communication_timeout="$(arg communication_timeout)"
     />
   </xacro:if>

File: kuka_kr_description/robots/kr210_r2700.urdf.xacro (robot description, xacro)
@@ -4,5 +4,6 @@
   <xacro:arg name="rsi_ip" default="127.0.0.1"/>
   <xacro:arg name="rsi_port" default="49152"/>
-  <xacro:arg name="socket_timeout" default="30"/>
+  <xacro:arg name="connection_timeout" default="30"/>
+  <xacro:arg name="communication_timeout" default="1"/>
   <xacro:arg name="has_ft_sensor" default="false"/>
   <xacro:arg name="load_ros2_control" default="false"/>
@@ -19,5 +20,6 @@
             rsi_ip="$(arg rsi_ip)"
             rsi_port="$(arg rsi_port)"
-            socket_timeout="$(arg socket_timeout)"
+            connection_timeout="$(arg connection_timeout)"
+            communication_timeout="$(arg communication_timeout)"
             has_ft_sensor="$(arg has_ft_sensor)"
     />

File: kuka_kr_description/robots/kr70.urdf.xacro (robot description, xacro)
@@ -4,5 +4,6 @@
   <xacro:arg name="rsi_ip" default="127.0.0.1"/>
   <xacro:arg name="rsi_port" default="49152"/>
-  <xacro:arg name="socket_timeout" default="30"/>
+  <xacro:arg name="connection_timeout" default="30"/>
+  <xacro:arg name="communication_timeout" default="1"/>
   <xacro:arg name="has_ft_sensor" default="false"/>
   <xacro:arg name="load_ros2_control" default="false"/>
@@ -19,5 +20,6 @@
             rsi_ip="$(arg rsi_ip)"
             rsi_port="$(arg rsi_port)"
-            socket_timeout="$(arg socket_timeout)"
+            connection_timeout="$(arg connection_timeout)"
+            communication_timeout="$(arg communication_timeout)"
             has_ft_sensor="$(arg has_ft_sensor)"
     />

File: kuka_kr_description/ros2_control/kr10_r1100_2.ros2_control.xacro (robot description, xacro)
@@ -1,5 +1,5 @@
 <?xml version="1.0"?>
 <robot xmlns:xacro="http://www.ros.org/wiki/xacro" name="kr10_r1100_2_ros2_control">
-  <xacro:macro name="kr10_r1100_2_interface" params="name prefix rsi_ip rsi_port socket_timeout has_ft_sensor">
+  <xacro:macro name="kr10_r1100_2_interface" params="name prefix rsi_ip rsi_port connection_timeout communication_timeout has_ft_sensor">
     <ros2_control name="${name}" type="system">
       <hardware>
@@ -7,5 +7,6 @@
         <param name="rsi_ip">${rsi_ip}</param>
         <param name="rsi_port">${rsi_port}</param>
-        <param name="socket_timeout">${socket_timeout}</param>
+        <param name="connection_timeout">${connection_timeout}</param>
+        <param name="communication_timeout">${communication_timeout}</param>
       </hardware>
       <joint name="${prefix}joint_a1">

File: kuka_kr_description/ros2_control/kr16.ros2_control.xacro (robot description, xacro)
@@ -1,5 +1,5 @@
 <?xml version="1.0"?>
 <robot xmlns:xacro="http://www.ros.org/wiki/xacro" name="kr16_ros2_control">
-  <xacro:macro name="kr16_interface" params="name prefix rsi_ip rsi_port socket_timeout has_ft_sensor">
+  <xacro:macro name="kr16_interface" params="name prefix rsi_ip rsi_port connection_timeout communication_timeout has_ft_sensor">
     <ros2_control name="${name}" type="system">
       <hardware>
@@ -7,5 +7,6 @@
         <param name="rsi_ip">${rsi_ip}</param>
         <param name="rsi_port">${rsi_port}</param>
-        <param name="socket_timeout">${socket_timeout}</param>
+        <param name="connection_timeout">${connection_timeout}</param>
+        <param name="communication_timeout">${communication_timeout}</param>
       </hardware>
       <joint name="${prefix}joint_a1">

File: kuka_kr_description/ros2_control/kr16_2.ros2_control.xacro (robot description, xacro)
@@ -1,5 +1,5 @@
 <?xml version="1.0"?>
 <robot xmlns:xacro="http://www.ros.org/wiki/xacro" name="kr16_2_ros2_control">
-  <xacro:macro name="kr16_2_interface" params="name prefix rsi_ip rsi_port socket_timeout">
+  <xacro:macro name="kr16_2_interface" params="name prefix rsi_ip rsi_port connection_timeout communication_timeout">
     <ros2_control name="${name}" type="system">
       <hardware>
@@ -7,5 +7,6 @@
         <param name="rsi_ip">${rsi_ip}</param>
         <param name="rsi_port">${rsi_port}</param>
-        <param name="socket_timeout">${socket_timeout}</param>
+        <param name="connection_timeout">${connection_timeout}</param>
+        <param name="communication_timeout">${communication_timeout}</param>
       </hardware>
       <joint name="${prefix}joint_a1">

File: kuka_kr_description/ros2_control/kr210_r2700.ros2_control.xacro (robot description, xacro)
@@ -1,5 +1,5 @@
 <?xml version="1.0"?>
 <robot xmlns:xacro="http://www.ros.org/wiki/xacro" name="kr210_r2700_ros2_control">
-  <xacro:macro name="kr210_r2700_interface" params="name prefix rsi_ip rsi_port socket_timeout has_ft_sensor">
+  <xacro:macro name="kr210_r2700_interface" params="name prefix rsi_ip rsi_port connection_timeout communication_timeout has_ft_sensor">
     <ros2_control name="${name}" type="system">
       <hardware>
@@ -7,5 +7,6 @@
         <param name="rsi_ip">${rsi_ip}</param>
         <param name="rsi_port">${rsi_port}</param>
-        <param name="socket_timeout">${socket_timeout}</param>
+        <param name="connection_timeout">${connection_timeout}</param>
+        <param name="communication_timeout">${communication_timeout}</param>
       </hardware>
       <joint name="${prefix}joint_a1">

File: kuka_kr_description/ros2_control/kr70.ros2_control.xacro (robot description, xacro)
@@ -1,5 +1,5 @@
 <?xml version="1.0"?>
 <robot xmlns:xacro="http://www.ros.org/wiki/xacro" name="kr70_ros2_control">
-  <xacro:macro name="kr70_interface" params="name prefix rsi_ip rsi_port socket_timeout has_ft_sensor">
+  <xacro:macro name="kr70_interface" params="name prefix rsi_ip rsi_port connection_timeout communication_timeout has_ft_sensor">
     <ros2_control name="${name}" type="system">
       <hardware>
@@ -7,5 +7,6 @@
         <param name="rsi_ip">${rsi_ip}</param>
         <param name="rsi_port">${rsi_port}</param>
-        <param name="socket_timeout">${socket_timeout}</param>
+        <param name="connection_timeout">${connection_timeout}</param>
+        <param name="communication_timeout">${communication_timeout}</param>
       </hardware>
       <joint name="${prefix}joint_a1">
