Commit message: feat: update colors

File: kuka_kr_description/robots/kr210_r2700.xacro (robot description, xacro)
@@ -4,4 +4,10 @@
     <!-- LINKS -->
     <!-- base link -->
+    <material name="black">
+      <color rgba="0.2 0.2 0.2 1"/>
+    </material>
+    <material name="orange">
+      <color rgba="0.945 0.359 0.098 1"/>
+    </material>
     <link name="${prefix}base_link">
       <visual>
@@ -10,7 +16,5 @@
           <mesh filename="package://kuka_kr_description/meshes/kr210_r2700/visual/base_link.stl" />
         </geometry>
-        <material name="">
-          <color rgba="0.75294 0.75294 0.75294 1"/>
-        </material>
+        <material name="black"/>
       </visual>
       <collision>
@@ -33,7 +37,5 @@
           <mesh filename="package://kuka_kr_description/meshes/kr210_r2700/visual/link_1.stl" />
         </geometry>
-        <material name="">
-          <color rgba="0.75294 0.75294 0.75294 1"/>
-        </material>
+        <material name="orange"/>
       </visual>
       <collision>
@@ -56,7 +58,5 @@
           <mesh filename="package://kuka_kr_description/meshes/kr210_r2700/visual/link_2.stl"/>
         </geometry>
-        <material name="">
-          <color rgba="0.75294 0.75294 0.75294 1"/>
-        </material>
+        <material name="orange"/>
       </visual>
       <collision>
@@ -79,7 +79,5 @@
           <mesh filename="package://kuka_kr_description/meshes/kr210_r2700/visual/link_3.stl" />
         </geometry>
-        <material name="">
-          <color rgba="0.75294 0.75294 0.75294 1"/>
-        </material>
+        <material name="orange"/>
       </visual>
       <inertial>
@@ -102,7 +100,5 @@
           <mesh filename="package://kuka_kr_description/meshes/kr210_r2700/visual/link_4.stl" />
         </geometry>
-        <material name="">
-          <color rgba="0.75294 0.75294 0.75294 1"/>
-        </material>
+        <material name="orange"/>
       </visual>
       <collision>
@@ -125,7 +121,5 @@
           <mesh filename="package://kuka_kr_description/meshes/kr210_r2700/visual/link_5.stl" />
         </geometry>
-        <material name="">
-          <color rgba="0.75294 0.75294 0.75294 1"/>
-        </material>
+        <material name="orange"/>
       </visual>
       <collision>
@@ -148,7 +142,5 @@
           <mesh filename="package://kuka_kr_description/meshes/kr210_r2700/visual/link_6.stl" />
         </geometry>
-        <material name="">
-          <color rgba="0.75294 0.75294 0.75294 1"/>
-        </material>
+        <material name="black"/>
       </visual>
       <collision>

Commit message: fix: kr210 joint limits

File: kuka_kr_description/robots/kr210_r2700.xacro (robot description, xacro)
@@ -164,5 +164,5 @@
       <child link="${prefix}link_1"/>
       <axis xyz="0 0 -1"/>
-      <limit effort="0" lower="${radians(-185)}" upper="${radians(185)}" velocity="${radians(123)}"/>
+      <limit effort="0" lower="${radians(-185)}" upper="${radians(185)}" velocity="${radians(120)}"/>
     </joint>
     <!-- joint 2 (A2) -->
@@ -180,5 +180,5 @@
       <child link="${prefix}link_3"/>
       <axis xyz="0 1 0"/>
-      <limit effort="0" lower="${radians(0)}" upper="${radians(138)}" velocity="${radians(112)}"/>
+      <limit effort="0" lower="${radians(-120)}" upper="${radians(168)}" velocity="${radians(112)}"/>
     </joint>
     <!-- joint 4 (A4) -->
@@ -188,5 +188,5 @@
       <child link="${prefix}link_4"/>
       <axis xyz="0 0 -1"/>
-      <limit effort="0" lower="${radians(-125)}" upper="${radians(125)}" velocity="${radians(172)}"/>
+      <limit effort="0" lower="${radians(-350)}" upper="${radians(350)}" velocity="${radians(179)}"/>
     </joint>
     <!-- joint 5 (A5) -->
@@ -204,5 +204,5 @@
       <child link="${prefix}link_6"/>
       <axis xyz="0 0 -1"/>
-      <limit effort="0" lower="${radians(-350)}" upper="${radians(350)}" velocity="${radians(219)}"/>
+      <limit effort="0" lower="${radians(-350)}" upper="${radians(350)}" velocity="${radians(220)}"/>
     </joint>
     <!-- END JOINTS -->

File: kuka_kr_description/ros2_control/kr210_r2700.ros2_control.xacro (robot description, xacro)
@@ -16,6 +16,6 @@
         </command_interface>
         <command_interface name="velocity">
-          <param name="min">${radians(-123)}</param>
-          <param name="max">${radians(123)}</param>
+          <param name="min">${radians(-120)}</param>
+          <param name="max">${radians(120)}</param>
         </command_interface>
         <state_interface name="position"/>
@@ -36,6 +36,6 @@
       <joint name="${prefix}joint_a3">
         <command_interface name="position">
-          <param name="min">0</param>
-          <param name="max">${radians(138)}</param>
+          <param name="min">${radians(-120)}</param>
+          <param name="max">${radians(168)}</param>
         </command_interface>
         <command_interface name="velocity">
@@ -48,10 +48,10 @@
       <joint name="${prefix}joint_a4">
         <command_interface name="position">
-          <param name="min">${radians(-125)}</param>
-          <param name="max">${radians(125)}</param>
+          <param name="min">${radians(-350)}</param>
+          <param name="max">${radians(350)}</param>
         </command_interface>
         <command_interface name="velocity">
-          <param name="min">${radians(-172)}</param>
-          <param name="max">${radians(172)}</param>
+          <param name="min">${radians(-179)}</param>
+          <param name="max">${radians(179)}</param>
         </command_interface>
         <state_interface name="position"/>
@@ -76,6 +76,6 @@
         </command_interface>
         <command_interface name="velocity">
-          <param name="min">${radians(-219)}</param>
-          <param name="max">${radians(219)}</param>
+          <param name="min">${radians(-220)}</param>
+          <param name="max">${radians(220)}</param>
         </command_interface>
         <state_interface name="position"/>
