Commit message: fix: joint

File: kuka_kr_description/robots/kr3_r540.xacro (robot description, xacro)
@@ -97,5 +97,5 @@
     <!-- joint 4 (A4) -->
     <joint name="${prefix}joint_a4" type="revolute">
-      <origin xyz="0.26 0 0.025" rpy="0 0 0"/>
+      <origin xyz="0.26 0 0.02" rpy="0 0 0"/>
       <parent link="${prefix}link_3"/>
       <child link="${prefix}link_4"/>
